File: protopedal/protopedal.kicad_pcb (KiCad board)
At the start: 2 copper layers, 184 x 50 mm, 38 parts, among them J1 Barrel_Jack_Switch, J10 Conn_01x03, J11 Conn_01x03, J12 Conn_01x03, J13 Conn_01x04, J14 Conn_01x02, J15 Conn_01x02, J16 Conn_01x02, J17 Conn_01x03, J18 Conn_01x03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

Commit message: more
Parts:
- moved R4 1.20 mm to (99.6, 38.2)
Changed lines of the file:
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@@
 	(footprint "Snapeda:STA_CF14_STP"
 		(layer "F.Cu")
-		(at 98.425 38.608 90)
+		(at 99.568 38.227 90)
 		(tags "CF14JT1K00 ")
 		(property "Reference" "R4"

Commit message: Fix omnidrive schematic; other things too
Parts:
- removed J6: Conn_01x03, Connector_PinHeader_2.54mm:PinHeader_1x03_P2.54mm_Vertical
- moved SW2 199.1 mm to (202.7, 56.0)
- moved SW6 193.2 mm to (188.1, 55.1)
- moved J12 179.4 mm to (208.7, 28.7)
- moved SW7 170.8 mm to (163.3, 54.9)
- moved SW3 165.7 mm to (176.0, 55.8)
- moved SW5 162.7 mm to (137.4, 54.9)
- moved J13 158.2 mm to (226.4, 72.0), turned to 180 degrees
- moved RV5 154.5 mm to (121.3, 60.1)
- moved J14 151.8 mm to (202.2, 74.4), turned to 90 degrees
- moved RV4 137.7 mm to (108.6, 60.0)
- moved SW4 136.5 mm to (151.4, 55.8)
- moved J18 131.1 mm to (186.1, 74.3), turned to 90 degrees
- moved J15 124.9 mm to (177.3, 74.0), turned to -90 degrees
- moved J19 103.5 mm to (160.7, 74.0), turned to 90 degrees
- moved J16 99.0 mm to (151.9, 73.8), turned to -90 degrees
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Other:
- board size 184 x 50 mm -> 184.2 x 53.1 mm
