File: protopedal/protopedal.kicad_sch (KiCad schematic)
At the start: 8 parts, among them J1 Barrel_Jack_Switch, J2 IN1, J3 Out1

Commit message: Add symbols for pin headers
Parts:
- added J10, J11, J12, J5, J6, J7, J8, J9: Conn_01x03, symbol Connector_Generic:Conn_01x03
- added J4: Batt, symbol Connector_Generic:Conn_01x02
- added RV1: 1K, Snapeda:TRIM_PT01-D115D-B104, symbol Device:R_Potentiometer
- added RV2: 10K, Snapeda:TRIM_PT01-D115D-B104, symbol Device:R_Potentiometer
- added RV3: 100K, Snapeda:TRIM_PT01-D115D-B104, symbol Device:R_Potentiometer
- added RV4: 500K, Snapeda:TO_3310Y, symbol Device:R_Potentiometer
- added RV5: 1M, Snapeda:TO_3310Y, symbol Device:R_Potentiometer

Commit message: fixed some stuff
Parts:
- J10, J11, J12, J5, J6, J7, J8, J9: footprint (none) -> Connector_PinHeader_2.54mm:PinHeader_1x03_P2.54mm_Vertical
- J4: footprint (none) -> Connector_PinHeader_2.54mm:PinHeader_1x02_P2.54mm_Vertical
- R1, R2: footprint (none) -> Snapeda:STA_CF14_STP
Changed lines of the file:
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@@
 			)
 		)
-		(property "Footprint" ""
+		(property "Footprint" "Connector_PinHeader_2.54mm:PinHeader_1x03_P2.54mm_Vertical"
 			(at 100.33 104.14 0)
 			(hide yes)
@@
 			)
 		)
-		(property "Footprint" ""
+		(property "Footprint" "Snapeda:STA_CF14_STP"
 			(at 68.072 35.56 90)
 			(hide yes)
@@
 			)
 		)
-		(property "Footprint" ""
+		(property "Footprint" "Connector_PinHeader_2.54mm:PinHeader_1x02_P2.54mm_Vertical"
 			(at 29.21 19.05 0)
 			(hide yes)
@@
 			)
 		)
-		(property "Footprint" ""
+		(property "Footprint" "Snapeda:STA_CF14_STP"
 			(at 94.742 38.1 90)
 			(hide yes)
@@
 			)
 		)
-		(property "Footprint" ""
+		(property "Footprint" "Connector_PinHeader_2.54mm:PinHeader_1x03_P2.54mm_Vertical"
 			(at 125.73 102.87 0)
 			(hide yes)
@@
 			)
 		)
-		(property "Footprint" ""
+		(property "Footprint" "Connector_PinHeader_2.54mm:PinHeader_1x03_P2.54mm_Vertical"
 			(at -7020.56 -863.6 0)
 			(hide yes)
@@
 			)
 		)
-		(property "Footprint" ""
+		(property "Footprint" "Connector_PinHeader_2.54mm:PinHeader_1x03_P2.54mm_Vertical"
 			(at 67.31 102.87 0)
 			(hide yes)
@@
 			)
 		)
-		(property "Footprint" ""
+		(property "Footprint" "Connector_PinHeader_2.54mm:PinHeader_1x03_P2.54mm_Vertical"
 			(at 152.4 102.87 0)
 			(hide yes)
@@
 			)
 		)
-		(property "Footprint" ""
+		(property "Footprint" "Connector_PinHeader_2.54mm:PinHeader_1x03_P2.54mm_Vertical"
 			(at 31.75 101.6 0)
 			(hide yes)
@@
 			)
 		)
-		(property "Footprint" ""
+		(property "Footprint" "Connector_PinHeader_2.54mm:PinHeader_1x03_P2.54mm_Vertical"
 			(at 242.57 71.12 0)
 			(hide yes)
@@
 			)
 		)
-		(property "Footprint" ""
+		(property "Footprint" "Connector_PinHeader_2.54mm:PinHeader_1x03_P2.54mm_Vertical"
 			(at 27.94 69.85 0)
 			(hide yes)

Commit message: started wiring
Parts:
- removed J4: Batt, Connector_PinHeader_2.54mm:PinHeader_1x02_P2.54mm_Vertical, symbol Connector_Generic:Conn_01x02
- added R3, R4: 100K, Snapeda:STA_CF14_STP, symbol Device:R
Connections:
- net at D5.1 (K): now also SW1.4
- net at D5.2 (A): now also R2.2
- net VCC: now reaches R1.1
- net VCC: now also J1.1, R2.1
- net at R1.2: now also D4.2 (A)
- net at SW1.8: now also J12.3 (Pin_3), J3.T
- net at SW1.9: now also J11.3 (Pin_3), J2.T, SW1.1
- net GND: now reaches SW1.5
- net GND: now also D4.1 (K), J1.2, J11.1 (Pin_1), J12.1 (Pin_1), J2.S, J3.S
- net at J3.R: now also J12.2 (Pin_2)
- net at J11.2 (Pin_2): now also J2.R
Other:
- moved on the sheet: D4, D5, J1, J11, J12, J2, J3, R1, R2, SW1A, SW1B, SW1C

Commit message: more
Parts:
- added C1: 10uF, Capacitor_THT:CP_Radial_D5.0mm_P2.00mm, symbol Device:C_Polarized_Small
- added J13: Conn_01x04, Connector_PinHeader_2.54mm:PinHeader_1x04_P2.54mm_Horizontal, symbol Connector_Generic:Conn_01x04
- added J14, J15, J16: Conn_01x02, symbol Connector_Generic:Conn_01x02
- added J17, J18, J19: Conn_01x03, symbol Connector_Generic:Conn_01x03
- added J4: Conn_01x04, Connector_PinHeader_2.54mm:PinHeader_1x04_P2.54mm_Vertical, symbol Connector_Generic:Conn_01x04
- added SW2, SW3, SW4: SW_SPST, symbol Switch:SW_SPST
- added SW5, SW6, SW7: SW_SPDT, symbol Switch:SW_SPDT
- SW1: footprint (none) -> SparkFun-Electromechanical:STOMP-SWITCH-3PDT
Connections:
- net GND: now also R3.2, C1.2, J13.1 (Pin_1), J4.1 (Pin_1)
- net VCC: now also R4.2, J13.2 (Pin_2), J4.2 (Pin_2)
- net at J8.1 (Pin_1): now also RV3.1
- net at J8.2 (Pin_2): now also RV3.2
- net at J8.3 (Pin_3): now also RV3.3
- net at RV1.1: now also J5.1 (Pin_1)
- net at RV1.2: now also J5.2 (Pin_2)
- net at RV1.3: now also J5.3 (Pin_3)
- net at J9.1 (Pin_1): now also RV4.1
- net at J9.2 (Pin_2): now also RV4.2
- net at J9.3 (Pin_3): now also RV4.3
- net INSIG: now reaches SW1.2
- net INSIG: now also J13.4 (Pin_4), J4.4 (Pin_4)
- net +4.5V: now reaches R4.1
- net +4.5V: now also R3.1, C1.1, J13.3 (Pin_3), J4.3 (Pin_3)
- net at J7.1 (Pin_1): now also RV2.1
- net at J7.2 (Pin_2): now also RV2.2
- net at J7.3 (Pin_3): now also RV2.3
- net at J10.1 (Pin_1): now also RV5.1
- net at J10.2 (Pin_2): now also RV5.2
- net at J10.3 (Pin_3): now also RV5.3
- new net: J16.1 (Pin_1), SW4.2 (B)
- new net: J16.2 (Pin_2), SW4.1 (A)
- new net: J17.1 (Pin_1), SW5.1 (A)
- new net: J17.2 (Pin_2), SW5.2 (B)
- new net: J17.3 (Pin_3), SW5.3 (C)
- new net: J18.1 (Pin_1), SW6.1 (A)
- new net: J18.2 (Pin_2), SW6.2 (B)
- new net: J18.3 (Pin_3), SW6.3 (C)
- new net: J14.2 (Pin_2), SW2.1 (A)
- new net: J14.1 (Pin_1), SW2.2 (B)
- new net: J15.1 (Pin_1), SW3.2 (B)
- new net: J15.2 (Pin_2), SW3.1 (A)
- new net: J19.1 (Pin_1), SW7.1 (A)
- new net: J19.2 (Pin_2), SW7.2 (B)
- new net: J19.3 (Pin_3), SW7.3 (C)
Other:
- moved on the sheet: J10, J5, J7, J8, J9, R3, RV1, RV2, RV3

Commit message: more
Parts:
- J13: footprint Connector_PinHeader_2.54mm:PinHeader_1x04_P2.54mm_Horizontal -> Connector_PinHeader_2.54mm:PinHeader_1x04_P2.54mm_Vertical
- J14, J15, J16: footprint (none) -> Connector_PinHeader_2.54mm:PinHeader_1x02_P2.54mm_Vertical
- J17, J18, J19: footprint (none) -> Connector_PinHeader_2.54mm:PinHeader_1x03_P2.54mm_Vertical
- SW2, SW3, SW4: footprint (none) -> Snapeda:SW2_GF-123-0054_CWI
- SW5, SW6, SW7: footprint (none) -> Snapeda:ASE1E-2M-10-Z_NDC
Changed lines of the file:
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@@
 			)
 		)
-		(property "Footprint" ""
+		(property "Footprint" "Connector_PinHeader_2.54mm:PinHeader_1x02_P2.54mm_Vertical"
 			(at 106.68 106.68 0)
 			(hide yes)
@@
 			)
 		)
-		(property "Footprint" ""
+		(property "Footprint" "Connector_PinHeader_2.54mm:PinHeader_1x03_P2.54mm_Vertical"
 			(at 69.85 128.27 0)
 			(hide yes)
@@
 			)
 		)
-		(property "Footprint" ""
+		(property "Footprint" "Snapeda:ASE1E-2M-10-Z_NDC"
 			(at 91.44 130.81 0)
 			(hide yes)
@@
 			)
 		)
-		(property "Footprint" ""
+		(property "Footprint" "Snapeda:SW2_GF-123-0054_CWI"
 			(at 76.2 99.06 0)
 			(hide yes)
@@
 			)
 		)
-		(property "Footprint" ""
+		(property "Footprint" "Connector_PinHeader_2.54mm:PinHeader_1x02_P2.54mm_Vertical"
 			(at 92.71 106.68 0)
 			(hide yes)
@@
 			)
 		)
-		(property "Footprint" ""
+		(property "Footprint" "Snapeda:ASE1E-2M-10-Z_NDC"
 			(at 130.81 130.81 0)
 			(hide yes)
@@
 			)
 		)
-		(property "Footprint" "Connector_PinHeader_2.54mm:PinHeader_1x04_P2.54mm_Horizontal"
+		(property "Footprint" "Connector_PinHeader_2.54mm:PinHeader_1x04_P2.54mm_Vertical"
 			(at 52.07 113.03 0)
 			(hide yes)
@@
 			)
 		)
-		(property "Footprint" ""
+		(property "Footprint" "Snapeda:ASE1E-2M-10-Z_NDC"
 			(at 53.34 128.27 0)
 			(hide yes)
@@
 			)
 		)
-		(property "Footprint" ""
+		(property "Footprint" "Connector_PinHeader_2.54mm:PinHeader_1x03_P2.54mm_Vertical"
 			(at 105.41 130.81 0)
 			(hide yes)
@@
 			)
 		)
-		(property "Footprint" ""
+		(property "Footprint" "Snapeda:SW2_GF-123-0054_CWI"
 			(at 105.41 99.06 0)
 			(hide yes)
@@
 			)
 		)
-		(property "Footprint" ""
+		(property "Footprint" "Connector_PinHeader_2.54mm:PinHeader_1x03_P2.54mm_Vertical"
 			(at 146.05 130.81 0)
 			(hide yes)
@@
 			)
 		)
-		(property "Footprint" ""
+		(property "Footprint" "Snapeda:SW2_GF-123-0054_CWI"
 			(at 91.44 99.06 0)
 			(hide yes)
@@
 			)
 		)
-		(property "Footprint" ""
+		(property "Footprint" "Connector_PinHeader_2.54mm:PinHeader_1x02_P2.54mm_Vertical"
 			(at 76.2 106.68 0)
 			(hide yes)

Commit message: Fix omnidrive schematic; other things too
Parts:
- removed J6: Conn_01x03, Connector_PinHeader_2.54mm:PinHeader_1x03_P2.54mm_Vertical, symbol Connector_Generic:Conn_01x03
Changed lines of the file:
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@@
-	(symbol
-		(lib_id "Connector_Generic:Conn_01x03")
-		(at -7020.56 -863.6 0)
-		(unit 1)
-		(body_style 1)
-		(exclude_from_sim no)
-		(in_bom yes)
-		(on_board yes)
-		(in_pos_files yes)
-		(dnp no)
-		(fields_autoplaced yes)
-		(property "Reference" "J6"
-			(at -7016.75 -864.8701 0)
-			(show_name no)
-			(do_not_autoplace no)
-			(effects
-				(font
-					(size 1.27 1.27)
-				)
-				(justify left)
-			)
-		)
-		(property "Value" "Conn_01x03"
-			(at -7016.75 -862.3301 0)
-			(show_name no)
-			(do_not_autoplace no)
-			(effects
-				(font
-					(size 1.27 1.27)
-				)
-				(justify left)
-			)
-		)
-		(property "Footprint" "Connector_PinHeader_2.54mm:PinHeader_1x03_P2.54mm_Vertical"
-			(at -7020.56 -863.6 0)
-			(hide yes)
-			(show_name no)
-			(do_not_autoplace no)
-			(effects
-				(font
-					(size 1.27 1.27)
-				)
-			)
-		)
-		(property "Datasheet" ""
-			(at -7020.56 -863.6 0)
-			(hide yes)
-			(show_name no)
-			(do_not_autoplace no)
-			(effects
-				(font
-					(size 1.27 1.27)
-				)
-			)
-		)
-		(property "Description" "Generic connector, single row, 01x03, script generated (kicad-library-utils/schlib/autogen/connector/)"
-			(at -7020.56 -863.6 0)
-			(hide yes)
-			(show_name no)
-			(do_not_autoplace no)
-			(effects
-				(font
-					(size 1.27 1.27)
-				)
-			)
-		)
-		(pin "2"
-		)
-		(pin "1"
-		)
-		(pin "3"
-		)
-		(instances
-			(project "protopedal"
-				(path "/e94a0a1e-667d-4e6b-839b-102ae72e5f6f"
-					(reference "J6")
-					(unit 1)
-				)
-			)
-		)
-	)
 	(symbol
 		(lib_id "Connector_Generic:Conn_01x03")
