File: easyvibe/easyvibe/easyvibe.kicad_sch (KiCad schematic)
At the start: 86 parts, among them SW1 SW_DPDT_x2, U1 TL062, U2 TL062, U3 TL062, U4 TL062

Commit message: Fix switch wiring
Connections:
- net GND: now also U3.4 (V-), U4.4 (V-)
- net at J_OUT1.T, J_OUT_TIP1.1 (Pin_1), J_STOMP_1.1 (Pin_1)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: now also J_STOMP6.1 (Pin_1), SW1.6 (C); no longer J_STOMP4.1 (Pin_1), SW1.4 (A)
- new net: J_STOMP4.1 (Pin_1), SW1.4 (A)
Changed lines of the file:
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@@
 	)
 	(junction
+		(at 271.78 24.13)
+		(diameter 0)
+		(color 0 0 0 0)
+	)
+	(junction
 		(at 259.08 93.98)
 		(diameter 0)
@@
 	)
 	(junction
+		(at 97.79 21.59)
+		(diameter 0)
+		(color 0 0 0 0)
+	)
+	(junction
 		(at 179.07 111.76)
 		(diameter 0)
@@
 	(wire
 		(pts
-			(xy 55.88 57.15) (xy 55.88 53.34)
+			(xy 48.26 111.76) (xy 48.26 120.65)
 		)
 		(stroke
@@
 	(wire
 		(pts
-			(xy 271.78 21.59) (xy 271.78 24.13)
+			(xy 55.88 57.15) (xy 55.88 53.34)
 		)
 		(stroke
@@
 	(wire
 		(pts
-			(xy 29.21 110.49) (xy 29.21 113.03)
+			(xy 271.78 21.59) (xy 271.78 24.13)
 		)
 		(stroke
@@
 	(wire
 		(pts
-			(xy 179.07 39.37) (xy 180.34 39.37)
+			(xy 29.21 110.49) (xy 29.21 113.03)
 		)
 		(stroke
@@
 	(wire
 		(pts
-			(xy 135.89 41.91) (xy 137.16 41.91)
+			(xy 179.07 39.37) (xy 180.34 39.37)
 		)
 		(stroke
@@
 	(wire
 		(pts
-			(xy 78.74 111.76) (xy 78.74 116.84)
+			(xy 135.89 41.91) (xy 137.16 41.91)
 		)
 		(stroke
@@
 	(wire
 		(pts
-			(xy 48.26 111.76) (xy 38.1 111.76)
+			(xy 78.74 111.76) (xy 78.74 116.84)
 		)
 		(stroke
@@
 	(wire
 		(pts
-			(xy 271.78 12.7) (xy 73.66 12.7)
-		)
-		(stroke
-			(width 0)
-			(type default)
-		)
-	)
-	(wire
-		(pts
 			(xy 137.16 36.83) (xy 137.16 30.48)
 		)
@@
 	(wire
 		(pts
+			(xy 214.63 24.13) (xy 271.78 24.13)
+		)
+		(stroke
+			(width 0)
+			(type default)
+		)
+	)
+	(wire
+		(pts
 			(xy 111.76 83.82) (xy 205.74 83.82)
 		)
@@
 	(wire
 		(pts
+			(xy 97.79 13.97) (xy 97.79 21.59)
+		)
+		(stroke
+			(width 0)
+			(type default)
+		)
+	)
+	(wire
+		(pts
 			(xy 88.9 124.46) (xy 99.06 124.46)
 		)
@@
 	(wire
 		(pts
+			(xy 214.63 24.13) (xy 214.63 13.97)
+		)
+		(stroke
+			(width 0)
+			(type default)
+		)
+	)
+	(wire
+		(pts
 			(xy 36.83 74.93) (xy 35.56 74.93)
 		)
@@
 	(wire
 		(pts
-			(xy 38.1 111.76) (xy 38.1 110.49)
-		)
-		(stroke
-			(width 0)
-			(type default)
-		)
-	)
-	(wire
-		(pts
 			(xy 222.25 87.63) (xy 222.25 88.9)
 		)
@@
 	(wire
 		(pts
+			(xy 97.79 21.59) (xy 73.66 21.59)
+		)
+		(stroke
+			(width 0)
+			(type default)
+		)
+	)
+	(wire
+		(pts
 			(xy 60.96 33.02) (xy 60.96 39.37)
 		)
@@
 	(wire
 		(pts
+			(xy 38.1 110.49) (xy 38.1 120.65)
+		)
+		(stroke
+			(width 0)
+			(type default)
+		)
+	)
+	(wire
+		(pts
 			(xy 39.37 57.15) (xy 55.88 57.15)
 		)
@@
 	(wire
 		(pts
+			(xy 214.63 13.97) (xy 97.79 13.97)
+		)
+		(stroke
+			(width 0)
+			(type default)
+		)
+	)
+	(wire
+		(pts
 			(xy 111.76 31.75) (xy 111.76 38.1)
 		)
@@
 	(wire
 		(pts
-			(xy 105.41 21.59) (xy 73.66 21.59)
+			(xy 105.41 21.59) (xy 97.79 21.59)
 		)
 		(stroke
@@
 	)
 	(symbol
+		(lib_id "power:GND")
+		(at 48.26 120.65 0)
+		(unit 1)
+		(body_style 1)
+		(exclude_from_sim no)
+		(in_bom yes)
+		(on_board yes)
+		(in_pos_files yes)
+		(dnp no)
+		(fields_autoplaced yes)
+		(property "Reference" "#PWR013"
+			(at 48.26 127 0)
+			(hide yes)
+			(show_name no)
+			(do_not_autoplace no)
+			(effects
+				(font
+					(size 1.27 1.27)
+				)
+			)
+		)
+		(property "Value" "GND"
+			(at 48.26 125.73 0)
+			(show_name no)
+			(do_not_autoplace no)
+			(effects
+				(font
+					(size 1.27 1.27)
+				)
+			)
+		)
+		(property "Footprint" ""
+			(at 48.26 120.65 0)
+			(hide yes)
+			(show_name no)
+			(do_not_autoplace no)
+			(effects
+				(font
+					(size 1.27 1.27)
+				)
+			)
+		)
+		(property "Datasheet" ""
+			(at 48.26 120.65 0)
+			(hide yes)
+			(show_name no)
+			(do_not_autoplace no)
+			(effects
+				(font
+					(size 1.27 1.27)
+				)
+			)
+		)
+		(property "Description" "Power symbol creates a global label with name \"GND\" , ground"
+			(at 48.26 120.65 0)
+			(hide yes)
+			(show_name no)
+			(do_not_autoplace no)
+			(effects
+				(font
+					(size 1.27 1.27)
+				)
+			)
+		)
+		(pin "1"
+		)
+		(instances
+			(project "easyvibe"
+				(path "/4bb4501e-45c8-4c72-91ca-8621e8761900"
+					(reference "#PWR013")
+					(unit 1)
+				)
+			)
+		)
+	)
+	(symbol
 		(lib_id "Device:D")
 		(at 78.74 107.95 270)
@@
 				)
 			)
+		)
+	)
+	(symbol
+		(lib_id "power:GND")
+		(at 38.1 120.65 0)
+		(unit 1)
+		(body_style 1)
+		(exclude_from_sim no)
+		(in_bom yes)
+		(on_board yes)
+		(in_pos_files yes)
+		(dnp no)
+		(fields_autoplaced yes)
+		(property "Reference" "#PWR012"
+			(at 38.1 127 0)
+			(hide yes)
+			(show_name no)
+			(do_not_autoplace no)
+			(effects
+				(font
+					(size 1.27 1.27)
+				)
+			)
+		)
+		(property "Value" "GND"
+			(at 38.1 125.73 0)
+			(show_name no)
+			(do_not_autoplace no)
+			(effects
+				(font
+					(size 1.27 1.27)
+				)
+			)
+		)
+		(property "Footprint" ""
+			(at 38.1 120.65 0)
+			(hide yes)
+			(show_name no)
+			(do_not_autoplace no)
+			(effects
+				(font
+					(size 1.27 1.27)
+				)
+			)
+		)
+		(property "Datasheet" ""
+			(at 38.1 120.65 0)
+			(hide yes)
+			(show_name no)
+			(do_not_autoplace no)
+			(effects
+				(font
+					(size 1.27 1.27)
+				)
+			)
+		)
+		(property "Description" "Power symbol creates a global label with name \"GND\" , ground"
+			(at 38.1 120.65 0)
+			(hide yes)
+			(show_name no)
+			(do_not_autoplace no)
+			(effects
+				(font
+					(size 1.27 1.27)
+				)
+			)
+		)
+		(pin "1"
+		)
+		(instances
+			(project "easyvibe"
+				(path "/4bb4501e-45c8-4c72-91ca-8621e8761900"
+					(reference "#PWR012")
+					(unit 1)
+				)
+			)
